File: PiezoPhone/_restore_backup_2026-07-01T14-12-37-191/PiezoPhone.kicad_pcb (KiCad board)
At the start: 2 copper layers, 74.7 x 100 mm, 57 parts, among them J1 Screw_Terminal_01x02, J2 Screw_Terminal_01x02, J3 Screw_Terminal_01x02, J4 Screw_Terminal_01x02, J5 Screw_Terminal_01x02, J6 Screw_Terminal_01x02, J7 Screw_Terminal_01x02, J8 SJ1-3525NG, J9 Conn_01x02_Socket, SW1 SW_DIP_x04, U1 LM386

Commit message: Update PCB v1.1
Other:
- board size 74.7 x 100 mm -> 74.7 x 100.6 mm
- board text added: "Digital Marimba version 1.0 R. Dunbar Poor"
- board text removed: "Digital Marimba version 1.1 R. Dunbar Poor"
Changed lines of the file:
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@@
 	)
 	(setup
-		(stackup
-			(layer "F.SilkS"
-				(type "Top Silk Screen")
-			)
-			(layer "F.Paste"
-				(type "Top Solder Paste")
-			)
-			(layer "F.Mask"
-				(type "Top Solder Mask")
-				(thickness 0.01)
-			)
-			(layer "F.Cu"
-				(type "copper")
-				(thickness 0.035)
-			)
-			(layer "dielectric 1"
-				(type "core")
-				(thickness 1.51)
-				(material "FR4")
-				(epsilon_r 4.5)
-				(loss_tangent 0.02)
-			)
-			(layer "B.Cu"
-				(type "copper")
-				(thickness 0.035)
-			)
-			(layer "B.Mask"
-				(type "Bottom Solder Mask")
-				(thickness 0.01)
-			)
-			(layer "B.Paste"
-				(type "Bottom Solder Paste")
-			)
-			(layer "B.SilkS"
-				(type "Bottom Silk Screen")
-			)
-			(copper_finish "None")
-			(dielectric_constraints no)
-		)
 		(pad_to_mask_clearance 0)
 		(allow_soldermask_bridges_in_footprints no)
@@
 		(pcbplotparams
 			(layerselection 0x00000000_00000000_55555555_5755f5ff)
-			(plot_on_all_layers_selection 0x00000000_00000000_00000000_02000000)
+			(plot_on_all_layers_selection 0x00000000_00000000_00000000_00000000)
 			(disableapertmacros no)
-			(usegerberextensions yes)
+			(usegerberextensions no)
 			(usegerberattributes yes)
 			(usegerberadvancedattributes yes)
-			(creategerberjobfile no)
+			(creategerberjobfile yes)
 			(dashed_line_dash_ratio 12)
 			(dashed_line_gap_ratio 3)
@@
 			(outputformat 1)
 			(mirror no)
-			(drillshape 0)
+			(drillshape 1)
 			(scaleselection 1)
-			(outputdirectory "jlcpcb_plots/")
+			(outputdirectory "")
 		)
 	)
@@
 		(tags "THT DIP DIL PDIP 2.54mm 7.62mm 300mil Socket")
 		(property "Reference" "SW1"
-			(at 10.85 -0.422 180)
+			(at 3.81 -2.33 0)
 			(layer "F.SilkS")
 			(effects
@@
 		(tags "connector JST PH horizontal")
 		(property "Reference" "J9"
-			(at 3.548 8.096 180)
+			(at 1 -2.55 90)
 			(layer "F.SilkS")
 			(effects
@@
 		(tags "Resistor Axial_DIN0411 series Axial Horizontal pin pitch 12.7mm 1W length 9.9mm diameter 3.6mm")
 		(property "Reference" "FB2"
-			(at 6.35 2.72 90)
+			(at 6.35 -2.92 90)
 			(layer "F.SilkS")
 			(effects
@@
 		(tags "CP Radial series Radial pin pitch 2.50mm diameter 5mm height 7mm Electrolytic Capacitor")
 		(property "Reference" "C15"
-			(at -3.384 -1.58 90)
+			(at 1.25 -3.75 90)
 			(layer "F.SilkS")
 			(effects
@@
 		(tags "SJ1-3525NG ")
 		(property "Reference" "J8"
-			(at 7.452 6.563999 0)
+			(at 0 0 270)
 			(unlocked yes)
 			(layer "F.SilkS")
@@
 		(tags "C Disc series Radial pin pitch 5.00mm diameter 4.7mm width 2.5mm Capacitor")
 		(property "Reference" "C14"
-			(at 2.264 2.124 90)
+			(at 2.5 -2.5 90)
 			(layer "F.SilkS")
 			(effects
@@
 	)
 	(gr_rect
-		(start 61.468 32.5)
-		(end 136.144 132.5)
+		(start 61.468 32.004)
+		(end 136.144 132.588)
 		(stroke
 			(width 0.1)
@@
 		(layer "Edge.Cuts")
 	)
-	(gr_text "Digital Marimba\nversion 1.1\nR. Dunbar Poor"
+	(gr_text "Digital Marimba\nversion 1.0\nR. Dunbar Poor"
 		(at 117.5 128.5 0)
 		(layer "F.SilkS")
@@
 	)
 	(segment
+		(start 127.5 87.5)
+		(end 127.495349 87.504651)
+		(width 0.25)
+		(layer "F.Cu")
+		(net "Net-(C16-Pad1)")
+	)
+	(segment
 		(start 127.495349 87.504651)
 		(end 120.815349 87.504651)
@@
 	)
 	(segment
+		(start 123.564002 76.548)
+		(end 123.564002 76.828002)
+		(width 0.25)
+		(layer "F.Cu")
+		(net "Net-(C17-Pad2)")
+	)
+	(segment
 		(start 109.55 124.46)
 		(end 111.76 124.46)
@@
 		(net "Net-(R8-Pad2)")
 	)
+	(segment
+		(start 118.618 112.522)
+		(end 118.522 112.522)
+		(width 0.25)
+		(layer "B.Cu")
+		(net "Net-(R8-Pad2)")
+	)
+	(segment
+		(start 118.522 112.522)
+		(end 118.5 112.5)
+		(width 0.25)
+		(layer "B.Cu")
+		(net "Net-(R8-Pad2)")
+	)
